File: elec/ssslidar_v0.1_main_board.brd (EAGLE design)
At the start: 29 x 39 mm, 62 parts, among them IC1 MIC5504-2.8YM5, IC2 MIC5504-2.8YM5, K1 BUTTON-2P-REINFORCE-3100060P1, P10 PIN_SMD_1X1.6, P11 PIN_SMD_1X1.6, P12 PIN_SMD_1X1.6, P14 PIN_SMD_1X1.6, P15 PIN_SMD_1X1.6, P2 PIN_SMD_1X1.6, P3 PIN_SMD_1X1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

Commit message: Routing done.
Parts:
- added U$3: (no value), Xevelabs:XEVELABS_LOGO_S
- LED2: device Xevelabs:D_0603_L -> Xevelabs:D_0603_N
- moved C3 18.7 mm to (26.4, 30.9), turned to 180 degrees
- moved C11 8.33 mm to (10.7, 31.3)
- moved C7 7.32 mm to (14.6, 31.3), turned to 0 degrees
- moved U2 6.90 mm to (12.4, 33.6)
- moved L2 6.89 mm to (9.70, 33.6)
- moved L1 6.06 mm to (7.85, 33.2), turned to 90 degrees
- moved D1 5.59 mm to (19.2, 31.3), turned to 0 degrees
- moved C6 4.37 mm to (6.80, 29.8)
- moved IC1 2.20 mm to (3.70, 29.8)
- moved C4 0.95 mm to (27.2, 24.1)
- moved IC2 0.95 mm to (27.2, 27.2)
- moved D2 0.67 mm to (11.3, 36.1), turned to 0 degrees
- moved R1 0.32 mm to (13.2, 35.9), turned to 90 degrees
- moved LED2 0.17 mm to (10.7, 36.1)
Connections:
- net DXL<MCU: now also U4.27; no longer U4.26
- net DXL>MCU: now also U4.26; no longer U4.27
Routing:
- net N$10: track 63.7 -> 84.0 mm, vias 3 -> 2
- net N$14: track 8.16 -> 25.5 mm, vias 1 -> 2
- net N$13: track 7.89 -> 24.8 mm, vias 1 -> 2
- net DXL<MCU: track 17.9 -> 32.2 mm
- net DXL>MCU: track 18.9 -> 32.4 mm
- net 5V_OUT: track 3.48 -> 13.1 mm, vias 2 -> 4
- net N$11: track 63.9 -> 73.0 mm
- net N$5: track 0.00 -> 6.58 mm
- net N$12: track 75.6 -> 81.2 mm
- net +12V: track 4.16 -> 8.98 mm
- net VEE: track 48.7 -> 52.7 mm
- net +5V: track 0.00 -> 3.90 mm
- net N$8: track 0.00 -> 2.10 mm
- net GND: track 22.0 -> 23.1 mm, vias 13 -> 34
- net N$9: track 54.3 -> 53.6 mm
- added copper zone on layer 16, net N$3
- added copper zone on layer 16, net N$6
Other:
- board text added: "!R"
- board text added: "+"
- board text added: "-"
- board text added: "1"
- board text added: "2"
- board text added: "20160908"
- board text added: "3"
- board text added: "A"
- board text added: "B"
- board text added: "C"
- board text added: "DXLD"
- board text added: "G"
- board text added: "I"
- board text added: "PWR"
- board text added: "SIG"
- board text added: "SSSLidar"
- board text added: "V"
- board text added: "V1.0"
