File: elec/ssslidar_v0.1_main_board.sch (EAGLE design)
At the start: 60 parts, among them IC1 MIC5504-2.8YM5, IC2 MIC5504-2.8YM5, K1 BUTTON-2P-REINFORCE-3100060P1, P10 PIN_SMD_1X1.6, P11 PIN_SMD_1X1.6, P12 PIN_SMD_1X1.6, P14 PIN_SMD_1X1.6, P15 PIN_SMD_1X1.6, P2 PIN_SMD_1X1.6, P3 PIN_SMD_1X1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

Commit message: Only power and cosmetics left
Parts:
- added R4, R6: TBD, Xevelabs:R0402
Connections:
- new net N$13: JP1.TXO, R4.2
- new net N$14: JP1.RXI, R6.2
- new net N$15: IC2.BYP
- net RXD: now also R6.1; no longer JP1.RXI
- net TXD: now also R4.1; no longer JP1.TXO
- net VDD: no longer R3.2
- net VEE: now also R3.2
Changed lines of the file:
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@@
 <part name="GND25" library="supply1" deviceset="GND" device=""/>
 <part name="GND27" library="supply1" deviceset="GND" device=""/>
-<part name="VDD12" library="supply1" deviceset="VDD" device=""/>
+<part name="SUPPLY4" library="supply2" deviceset="VEE" device=""/>
+<part name="R4" library="Xevelabs" deviceset="R" device="0402" value="TBD"/>
+<part name="R6" library="Xevelabs" deviceset="R" device="0402" value="TBD"/>
 </parts>
 <sheets>
@@
 <instance part="C3" gate="G$1" x="78.74" y="226.06"/>
 <instance part="C4" gate="G$1" x="137.16" y="228.6"/>
-<instance part="P+2" gate="1" x="60.96" y="162.56"/>
+<instance part="P+2" gate="1" x="73.66" y="162.56"/>
 <instance part="GND12" gate="1" x="55.88" y="144.78"/>
 <instance part="JP1" gate="G$1" x="30.48" y="157.48" rot="MR0"/>
@@
 <instance part="GND25" gate="1" x="12.7" y="88.9"/>
 <instance part="GND27" gate="1" x="96.52" y="91.44"/>
-<instance part="VDD12" gate="G$1" x="68.58" y="30.48"/>
+<instance part="SUPPLY4" gate="G$1" x="68.58" y="30.48"/>
+<instance part="R4" gate="G$1" x="45.72" y="160.02" rot="R90"/>
+<instance part="R6" gate="G$1" x="45.72" y="157.48" rot="MR270"/>
 </instances>
 <busses>
@@
 <pinref part="VDD8" gate="G$1" pin="VDD"/>
 </segment>
-<segment>
-<pinref part="R3" gate="G$1" pin="2"/>
-<wire x1="68.58" y1="27.94" x2="68.58" y2="25.4" width="0.1524" layer="91"/>
-<pinref part="VDD12" gate="G$1" pin="VDD"/>
-</segment>
 </net>
 <net name="C_INT2" class="0">
@@
 <wire x1="243.84" y1="45.72" x2="243.84" y2="53.34" width="0.1524" layer="91"/>
 <junction x="243.84" y="53.34"/>
+<junction x="243.84" y="45.72"/>
 </segment>
 <segment>
@@
 <net name="+5V" class="0">
 <segment>
-<wire x1="35.56" y1="154.94" x2="60.96" y2="154.94" width="0.1524" layer="91"/>
+<wire x1="35.56" y1="154.94" x2="73.66" y2="154.94" width="0.1524" layer="91"/>
 <pinref part="P+2" gate="1" pin="+5V"/>
-<wire x1="60.96" y1="154.94" x2="60.96" y2="160.02" width="0.1524" layer="91"/>
+<wire x1="73.66" y1="154.94" x2="73.66" y2="160.02" width="0.1524" layer="91"/>
 <pinref part="JP1" gate="G$1" pin="VCC"/>
 </segment>
@@
 <net name="RXD" class="0">
 <segment>
-<wire x1="35.56" y1="157.48" x2="45.72" y2="157.48" width="0.1524" layer="91"/>
-<label x="45.72" y="157.48" size="1.778" layer="95"/>
-<pinref part="JP1" gate="G$1" pin="RXI"/>
+<label x="60.96" y="157.48" size="1.778" layer="95"/>
+<pinref part="R6" gate="G$1" pin="1"/>
+<wire x1="50.8" y1="157.48" x2="60.96" y2="157.48" width="0.1524" layer="91"/>
 </segment>
 <segment>
@@
 <net name="TXD" class="0">
 <segment>
-<wire x1="35.56" y1="160.02" x2="45.72" y2="160.02" width="0.1524" layer="91"/>
-<label x="45.72" y="160.02" size="1.778" layer="95"/>
-<pinref part="JP1" gate="G$1" pin="TXO"/>
+<label x="60.96" y="160.02" size="1.778" layer="95"/>
+<pinref part="R4" gate="G$1" pin="1"/>
+<wire x1="50.8" y1="160.02" x2="60.96" y2="160.02" width="0.1524" layer="91"/>
 </segment>
 <segment>
@@
 <wire x1="157.48" y1="15.24" x2="177.8" y2="15.24" width="0.1524" layer="91"/>
 <pinref part="SUPPLY5" gate="G$1" pin="VEE"/>
+</segment>
+<segment>
+<pinref part="R3" gate="G$1" pin="2"/>
+<wire x1="68.58" y1="27.94" x2="68.58" y2="25.4" width="0.1524" layer="91"/>
+<pinref part="SUPPLY4" gate="G$1" pin="VEE"/>
 </segment>
 </net>
@@
 </segment>
 </net>
+<net name="N$13" class="0">
+<segment>
+<pinref part="R4" gate="G$1" pin="2"/>
+<wire x1="35.56" y1="160.02" x2="40.64" y2="160.02" width="0.1524" layer="91"/>
+<pinref part="JP1" gate="G$1" pin="TXO"/>
+</segment>
+</net>
+<net name="N$14" class="0">
+<segment>
+<pinref part="R6" gate="G$1" pin="2"/>
+<wire x1="35.56" y1="157.48" x2="40.64" y2="157.48" width="0.1524" layer="91"/>
+<pinref part="JP1" gate="G$1" pin="RXI"/>
+</segment>
+</net>
+<net name="N$15" class="0">
+<segment>
+<pinref part="IC2" gate="G1" pin="BYP"/>
+<wire x1="93.98" y1="226.06" x2="91.44" y2="226.06" width="0.1524" layer="91"/>
+</segment>
+</net>

Commit message: Routing done.
Parts:
- LED2: device Xevelabs:LED0603_L -> Xevelabs:LED0603
Connections:
- net DXL<MCU: now also U4.PB4; no longer U4.PB3
- net DXL>MCU: now also U4.PB3; no longer U4.PB4
Changed lines of the file:
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@@
 <part name="D1" library="OPL" deviceset="D*" device="-SOD-123"/>
 <part name="L1" library="Xevelabs" deviceset="L" device="0603" value="Ferrite 10R BLM18BA100SN1D"/>
-<part name="LED2" library="Xevelabs" deviceset="LED" device="0603_L" value="Blue"/>
+<part name="LED2" library="Xevelabs" deviceset="LED" device="0603" value="Blue"/>
 <part name="R1" library="Xevelabs" deviceset="R" device="0402" value="470"/>
 <part name="GND15" library="supply1" deviceset="GND" device=""/>
@@
 </segment>
 <segment>
+<wire x1="264.16" y1="167.64" x2="269.24" y2="167.64" width="0.1524" layer="91"/>
+<label x="269.24" y="167.64" size="1.778" layer="95"/>
+<pinref part="U4" gate="A" pin="PB3"/>
+</segment>
+</net>
+<net name="DXL&lt;MCU" class="0">
+<segment>
+<pinref part="JP3" gate="G$1" pin="2"/>
+<wire x1="35.56" y1="127" x2="40.64" y2="127" width="0.1524" layer="91"/>
+<label x="40.64" y="127" size="1.778" layer="95"/>
+</segment>
+<segment>
 <wire x1="264.16" y1="165.1" x2="269.24" y2="165.1" width="0.1524" layer="91"/>
 <label x="269.24" y="165.1" size="1.778" layer="95"/>
@@
 </segment>
 </net>
-<net name="DXL&lt;MCU" class="0">
-<segment>
-<pinref part="JP3" gate="G$1" pin="2"/>
-<wire x1="35.56" y1="127" x2="40.64" y2="127" width="0.1524" layer="91"/>
-<label x="40.64" y="127" size="1.778" layer="95"/>
-</segment>
-<segment>
-<wire x1="264.16" y1="167.64" x2="269.24" y2="167.64" width="0.1524" layer="91"/>
-<label x="269.24" y="167.64" size="1.778" layer="95"/>
-<pinref part="U4" gate="A" pin="PB3"/>
-</segment>
-</net>
