File: elec/ssslidar_v1.0_main_board.sch (EAGLE design)
At the start: 61 parts, among them IC1 MIC5504-2.8YM5, IC2 MIC5504-2.8YM5, J1 DXLD_EXT_W_HOLES, K1 BUTTON-2P-REINFORCE-3100060P1, P10 PIN_SMD_1X1.6, P11 PIN_SMD_1X1.6, P12 PIN_SMD_1X1.6, P14 PIN_SMD_1X1.6, P15 PIN_SMD_1X1.6, P2 PIN_SMD_1X1.6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

Commit message: Finalized V1.0.
Connections:
- net DXL<MCU: now also J1.10
- net DXL>MCU: now also J1.9
Other:
- note removed: "TODO"
- moved on the sheet: J1, K1, L1
Changed lines of the file:
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@@
 <wire x1="271.78" y1="-30.48" x2="411.48" y2="-30.48" width="0.1524" layer="97"/>
 <text x="274.32" y="30.48" size="1.778" layer="97">Accel / Gyro</text>
-<text x="58.42" y="124.46" size="5.08" layer="92" rot="R90">TODO</text>
 </plain>
 <instances>
@@
 <instance part="P2" gate="G$1" x="142.24" y="154.94"/>
 <instance part="P3" gate="G$1" x="142.24" y="127"/>
-<instance part="GND21" gate="1" x="12.7" y="127"/>
+<instance part="GND21" gate="1" x="30.48" y="127"/>
 <instance part="U$2" gate="G$1" x="134.62" y="76.2" rot="MR0"/>
 <instance part="VDD6" gate="G$1" x="114.3" y="101.6"/>
@@
 <instance part="D2" gate="D" x="30.48" y="236.22"/>
 <instance part="P+1" gate="1" x="20.32" y="241.3"/>
-<instance part="L1" gate="G$1" x="20.32" y="142.24" rot="R180"/>
+<instance part="L1" gate="G$1" x="43.18" y="142.24" rot="R180"/>
 <instance part="LED2" gate="G$1" x="50.8" y="218.44"/>
 <instance part="R1" gate="G$1" x="50.8" y="208.28" rot="R180"/>
@@
 <instance part="R9" gate="G$1" x="299.72" y="48.26" rot="R270"/>
 <instance part="SUPPLY5" gate="G$1" x="177.8" y="17.78"/>
-<instance part="K1" gate="K" x="299.72" y="208.28"/>
-<instance part="GND18" gate="1" x="309.88" y="187.96"/>
+<instance part="K1" gate="K" x="304.8" y="208.28"/>
+<instance part="GND18" gate="1" x="314.96" y="198.12"/>
 <instance part="C1" gate="G$1" x="12.7" y="93.98"/>
 <instance part="C5" gate="G$1" x="96.52" y="96.52"/>
@@
 <instance part="C12" gate="G$1" x="304.8" y="-7.62"/>
 <instance part="GND38" gate="1" x="314.96" y="-12.7"/>
-<instance part="J1" gate="G$1" x="40.64" y="134.62"/>
-<instance part="P+3" gate="1" x="20.32" y="152.4"/>
+<instance part="J1" gate="G$1" x="63.5" y="134.62"/>
+<instance part="P+3" gate="1" x="43.18" y="152.4"/>
 <instance part="C7" gate="G$1" x="71.12" y="228.6"/>
 <instance part="C11" gate="G$1" x="71.12" y="195.58"/>
@@
 </segment>
 <segment>
-<wire x1="27.94" y1="134.62" x2="12.7" y2="134.62" width="0.1524" layer="91"/>
-<wire x1="12.7" y1="134.62" x2="12.7" y2="129.54" width="0.1524" layer="91"/>
+<wire x1="50.8" y1="134.62" x2="30.48" y2="134.62" width="0.1524" layer="91"/>
+<wire x1="30.48" y1="134.62" x2="30.48" y2="129.54" width="0.1524" layer="91"/>
 <pinref part="GND21" gate="1" pin="GND"/>
 <pinref part="J1" gate="G$1" pin="GND"/>
@@
 <segment>
 <pinref part="K1" gate="K" pin="2"/>
-<wire x1="307.34" y1="205.74" x2="309.88" y2="203.2" width="0.1524" layer="91"/>
-<wire x1="309.88" y1="203.2" x2="309.88" y2="190.5" width="0.1524" layer="91"/>
+<wire x1="312.42" y1="205.74" x2="314.96" y2="205.74" width="0.1524" layer="91"/>
+<wire x1="314.96" y1="205.74" x2="314.96" y2="200.66" width="0.1524" layer="91"/>
 <pinref part="GND18" gate="1" pin="GND"/>
-<wire x1="309.88" y1="203.2" x2="309.88" y2="208.28" width="0.1524" layer="91"/>
+<wire x1="314.96" y1="205.74" x2="314.96" y2="210.82" width="0.1524" layer="91"/>
 <pinref part="K1" gate="K" pin="S2"/>
-<wire x1="309.88" y1="208.28" x2="307.34" y2="210.82" width="0.1524" layer="91"/>
+<wire x1="314.96" y1="210.82" x2="312.42" y2="210.82" width="0.1524" layer="91"/>
 <pinref part="K1" gate="K" pin="S1"/>
-<wire x1="292.1" y1="210.82" x2="289.56" y2="210.82" width="0.1524" layer="91"/>
-<wire x1="289.56" y1="210.82" x2="289.56" y2="215.9" width="0.1524" layer="91"/>
-<wire x1="289.56" y1="215.9" x2="309.88" y2="215.9" width="0.1524" layer="91"/>
-<wire x1="309.88" y1="215.9" x2="309.88" y2="208.28" width="0.1524" layer="91"/>
-<junction x="309.88" y="203.2"/>
-<junction x="309.88" y="208.28"/>
+<wire x1="297.18" y1="210.82" x2="294.64" y2="210.82" width="0.1524" layer="91"/>
+<wire x1="294.64" y1="210.82" x2="294.64" y2="215.9" width="0.1524" layer="91"/>
+<wire x1="294.64" y1="215.9" x2="314.96" y2="215.9" width="0.1524" layer="91"/>
+<wire x1="314.96" y1="215.9" x2="314.96" y2="210.82" width="0.1524" layer="91"/>
+<junction x="314.96" y="205.74"/>
+<junction x="314.96" y="210.82"/>
 </segment>
 <segment>
@@
 <pinref part="P+3" gate="1" pin="+5V"/>
 <pinref part="L1" gate="G$1" pin="2"/>
-<wire x1="20.32" y1="147.32" x2="20.32" y2="149.86" width="0.1524" layer="91"/>
+<wire x1="43.18" y1="147.32" x2="43.18" y2="149.86" width="0.1524" layer="91"/>
 </segment>
 </net>
@@
 <net name="DXL&gt;MCU" class="0">
 <segment>
-<wire x1="60.96" y1="132.08" x2="66.04" y2="132.08" width="0.1524" layer="91"/>
-<label x="66.04" y="132.08" size="1.778" layer="95"/>
+<wire x1="50.8" y1="129.54" x2="43.18" y2="129.54" width="0.1524" layer="91"/>
+<label x="43.18" y="129.54" size="1.778" layer="95" rot="MR0"/>
+<pinref part="J1" gate="G$1" pin="9"/>
 </segment>
 <segment>
@@
 <net name="DXL&lt;MCU" class="0">
 <segment>
-<wire x1="60.96" y1="134.62" x2="66.04" y2="134.62" width="0.1524" layer="91"/>
-<label x="66.04" y="134.62" size="1.778" layer="95"/>
+<wire x1="76.2" y1="129.54" x2="83.82" y2="129.54" width="0.1524" layer="91"/>
+<label x="83.82" y="129.54" size="1.778" layer="95"/>
+<pinref part="J1" gate="G$1" pin="10"/>
 </segment>
 <segment>
@@
 <pinref part="K1" gate="K" pin="1"/>
 <pinref part="U4" gate="A" pin="PA4"/>
-<wire x1="292.1" y1="205.74" x2="264.16" y2="205.74" width="0.1524" layer="91"/>
+<wire x1="297.18" y1="205.74" x2="264.16" y2="205.74" width="0.1524" layer="91"/>
 </segment>
 </net>
@@
 <segment>
 <pinref part="J1" gate="G$1" pin="5V"/>
-<wire x1="27.94" y1="132.08" x2="20.32" y2="132.08" width="0.1524" layer="91"/>
-<wire x1="20.32" y1="132.08" x2="20.32" y2="137.16" width="0.1524" layer="91"/>
+<wire x1="50.8" y1="132.08" x2="43.18" y2="132.08" width="0.1524" layer="91"/>
+<wire x1="43.18" y1="132.08" x2="43.18" y2="137.16" width="0.1524" layer="91"/>
 <pinref part="L1" gate="G$1" pin="1"/>
 </segment>
