File: elec/ssslidar_v1.0_blade_PWR_top.sch (EAGLE design)
At the start: 24 parts, among them P1 PIN_SMD_0.8X1_RECT, P10 PIN_SMD_0.8X1_RECT, P11 PIN_SMD_1X1_RECT, P12 PIN_SMD_0.8X1_RECT, P13 PIN_SMD_0.8X1_RECT, P14 PIN_SMD_0.8X1_RECT, P16 PIN_SMD_0.8X1_RECT, P17 PIN_SMD_1X1_RECT, P18 PIN_SMD_0.8X1_RECT, P2 PIN_SMD_1X1_RECT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

Commit message: Upadted blade footprint, put everything in v1.0
Parts:
- P10, P12, P13, P16: value PIN_SMD_0.8X1_RECT -> PIN_SMD_1X1_RECT; device Xevelabs:PIN_SMD_0.8X1_RECT -> Xevelabs:PIN_SMD_1X1_RECT
Changed lines of the file:
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@@
 <grid distance="0.1" unitdist="inch" unit="inch" style="lines" multiple="1" display="no" altdistance="0.01" altunitdist="inch" altunit="inch"/>
 <layers>
-<layer number="1" name="Top" color="4" fill="1" visible="no" active="no"/>
-<layer number="2" name="Route2" color="1" fill="3" visible="no" active="no"/>
-<layer number="3" name="Route3" color="4" fill="3" visible="no" active="no"/>
-<layer number="14" name="Route14" color="1" fill="6" visible="no" active="no"/>
-<layer number="15" name="Route15" color="4" fill="6" visible="no" active="no"/>
-<layer number="16" name="Bottom" color="1" fill="1" visible="no" active="no"/>
-<layer number="17" name="Pads" color="2" fill="1" visible="no" active="no"/>
-<layer number="18" name="Vias" color="2" fill="1" visible="no" active="no"/>
-<layer number="19" name="Unrouted" color="6" fill="1" visible="no" active="no"/>
-<layer number="20" name="Dimension" color="15" fill="1" visible="no" active="no"/>
-<layer number="21" name="tPlace" color="7" fill="1" visible="no" active="no"/>
-<layer number="22" name="bPlace" color="7" fill="1" visible="no" active="no"/>
-<layer number="23" name="tOrigins" color="15" fill="1" visible="no" active="no"/>
-<layer number="24" name="bOrigins" color="15" fill="1" visible="no" active="no"/>
-<layer number="25" name="tNames" color="7" fill="1" visible="no" active="no"/>
-<layer number="26" name="bNames" color="7" fill="1" visible="no" active="no"/>
-<layer number="27" name="tValues" color="7" fill="1" visible="no" active="no"/>
-<layer number="28" name="bValues" color="7" fill="1" visible="no" active="no"/>
+<layer number="1" name="Top" color="4" fill="1" visible="yes" active="no"/>
+<layer number="2" name="Route2" color="1" fill="3" visible="yes" active="no"/>
+<layer number="3" name="Route3" color="4" fill="3" visible="yes" active="no"/>
+<layer number="14" name="Route14" color="1" fill="6" visible="yes" active="no"/>
+<layer number="15" name="Route15" color="4" fill="6" visible="yes" active="no"/>
+<layer number="16" name="Bottom" color="1" fill="1" visible="yes" active="no"/>
+<layer number="17" name="Pads" color="2" fill="1" visible="yes" active="no"/>
+<layer number="18" name="Vias" color="2" fill="1" visible="yes" active="no"/>
+<layer number="19" name="Unrouted" color="6" fill="1" visible="yes" active="no"/>
+<layer number="20" name="Dimension" color="15" fill="1" visible="yes" active="no"/>
+<layer number="21" name="tPlace" color="7" fill="1" visible="yes" active="no"/>
+<layer number="22" name="bPlace" color="7" fill="1" visible="yes" active="no"/>
+<layer number="23" name="tOrigins" color="15" fill="1" visible="yes" active="no"/>
+<layer number="24" name="bOrigins" color="15" fill="1" visible="yes" active="no"/>
+<layer number="25" name="tNames" color="7" fill="1" visible="yes" active="no"/>
+<layer number="26" name="bNames" color="7" fill="1" visible="yes" active="no"/>
+<layer number="27" name="tValues" color="7" fill="1" visible="yes" active="no"/>
+<layer number="28" name="bValues" color="7" fill="1" visible="yes" active="no"/>
 <layer number="29" name="tStop" color="7" fill="3" visible="no" active="no"/>
 <layer number="30" name="bStop" color="7" fill="6" visible="no" active="no"/>
@@
 <layer number="35" name="tGlue" color="7" fill="4" visible="no" active="no"/>
 <layer number="36" name="bGlue" color="7" fill="5" visible="no" active="no"/>
-<layer number="37" name="tTest" color="7" fill="1" visible="no" active="no"/>
-<layer number="38" name="bTest" color="7" fill="1" visible="no" active="no"/>
+<layer number="37" name="tTest" color="7" fill="1" visible="yes" active="no"/>
+<layer number="38" name="bTest" color="7" fill="1" visible="yes" active="no"/>
 <layer number="39" name="tKeepout" color="4" fill="11" visible="no" active="no"/>
 <layer number="40" name="bKeepout" color="1" fill="11" visible="no" active="no"/>
@@
 <layer number="44" name="Drills" color="7" fill="1" visible="no" active="no"/>
 <layer number="45" name="Holes" color="7" fill="1" visible="no" active="no"/>
-<layer number="46" name="Milling" color="3" fill="1" visible="no" active="no"/>
-<layer number="47" name="Measures" color="7" fill="1" visible="no" active="no"/>
-<layer number="48" name="Document" color="7" fill="1" visible="no" active="no"/>
-<layer number="49" name="Reference" color="7" fill="1" visible="no" active="no"/>
-<layer number="50" name="dxf" color="7" fill="1" visible="no" active="no"/>
-<layer number="51" name="tDocu" color="7" fill="1" visible="no" active="no"/>
-<layer number="52" name="bDocu" color="7" fill="1" visible="no" active="no"/>
-<layer number="53" name="tGND_GNDA" color="7" fill="9" visible="no" active="no"/>
-<layer number="54" name="bGND_GNDA" color="1" fill="9" visible="no" active="no"/>
-<layer number="56" name="wert" color="7" fill="1" visible="no" active="no"/>
+<layer number="46" name="Milling" color="3" fill="1" visible="yes" active="no"/>
+<layer number="47" name="Measures" color="7" fill="1" visible="yes" active="no"/>
+<layer number="48" name="Document" color="7" fill="1" visible="yes" active="no"/>
+<layer number="49" name="Reference" color="7" fill="1" visible="yes" active="no"/>
+<layer number="50" name="dxf" color="7" fill="1" visible="yes" active="no"/>
+<layer number="51" name="tDocu" color="7" fill="1" visible="yes" active="no"/>
+<layer number="52" name="bDocu" color="7" fill="1" visible="yes" active="no"/>
+<layer number="53" name="tGND_GNDA" color="7" fill="9" visible="yes" active="no"/>
+<layer number="54" name="bGND_GNDA" color="1" fill="9" visible="yes" active="no"/>
+<layer number="56" name="wert" color="7" fill="1" visible="yes" active="no"/>
 <layer number="90" name="Modules" color="5" fill="1" visible="yes" active="yes"/>
 <layer number="91" name="Nets" color="2" fill="1" visible="yes" active="yes"/>
@@
 <part name="P6" library="Xevelabs" deviceset="PIN" device="_SMD_0.8X1_RECT" value="PIN_SMD_0.8X1_RECT"/>
 <part name="P7" library="Xevelabs" deviceset="PIN" device="_SMD_0.8X1_RECT" value="PIN_SMD_0.8X1_RECT"/>
-<part name="P16" library="Xevelabs" deviceset="PIN" device="_SMD_0.8X1_RECT" value="PIN_SMD_0.8X1_RECT"/>
+<part name="P16" library="Xevelabs" deviceset="PIN" device="_SMD_1X1_RECT" value="PIN_SMD_1X1_RECT"/>
 <part name="P17" library="Xevelabs" deviceset="PIN" device="_SMD_1X1_RECT" value="PIN_SMD_1X1_RECT"/>
 <part name="P18" library="Xevelabs" deviceset="PIN" device="_SMD_0.8X1_RECT" value="PIN_SMD_0.8X1_RECT"/>
 <part name="P8" library="Xevelabs" deviceset="PIN" device="_SMD_0.8X1_RECT" value="PIN_SMD_0.8X1_RECT"/>
 <part name="P9" library="Xevelabs" deviceset="PIN" device="_SMD_1X1_RECT" value="PIN_SMD_1X1_RECT"/>
-<part name="P10" library="Xevelabs" deviceset="PIN" device="_SMD_0.8X1_RECT" value="PIN_SMD_0.8X1_RECT"/>
+<part name="P10" library="Xevelabs" deviceset="PIN" device="_SMD_1X1_RECT" value="PIN_SMD_1X1_RECT"/>
 <part name="P11" library="Xevelabs" deviceset="PIN" device="_SMD_1X1_RECT" value="PIN_SMD_1X1_RECT"/>
-<part name="P12" library="Xevelabs" deviceset="PIN" device="_SMD_0.8X1_RECT" value="PIN_SMD_0.8X1_RECT"/>
-<part name="P13" library="Xevelabs" deviceset="PIN" device="_SMD_0.8X1_RECT" value="PIN_SMD_0.8X1_RECT"/>
+<part name="P12" library="Xevelabs" deviceset="PIN" device="_SMD_1X1_RECT" value="PIN_SMD_1X1_RECT"/>
+<part name="P13" library="Xevelabs" deviceset="PIN" device="_SMD_1X1_RECT" value="PIN_SMD_1X1_RECT"/>
 <part name="R1" library="Xevelabs" deviceset="R" device="0402" value="2k"/>
 <part name="R2" library="Xevelabs" deviceset="R" device="0402" value="2k"/>

Commit message: Separated blades into bottom and top, since the bottom ones need to be taller to avoid seeing the Main PCB, or the screws...
Parts:
- removed P1, P18: PIN_SMD_0.8X1_RECT, Xevelabs:PIN_SMD_0.8X1_RECT
- P11, P17: value PIN_SMD_1X1_RECT -> PIN_SMD_1X2; device Xevelabs:PIN_SMD_1X1_RECT -> Xevelabs:PIN_SMD_1X2
Connections:
- removed net VDD_PASS: P1.1, P14.1
- net SCL: no longer P18.1
Other:
- moved on the sheet: P14
Changed lines of the file:
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@@
 <part name="VDD3" library="supply1" deviceset="VDD" device=""/>
 <part name="VDD4" library="supply1" deviceset="VDD" device=""/>
-<part name="P1" library="Xevelabs" deviceset="PIN" device="_SMD_0.8X1_RECT" value="PIN_SMD_0.8X1_RECT"/>
 <part name="P2" library="Xevelabs" deviceset="PIN" device="_SMD_1X1_RECT" value="PIN_SMD_1X1_RECT"/>
 <part name="P3" library="Xevelabs" deviceset="PIN" device="_SMD_0.8X1_RECT" value="PIN_SMD_0.8X1_RECT"/>
@@
 <part name="P7" library="Xevelabs" deviceset="PIN" device="_SMD_0.8X1_RECT" value="PIN_SMD_0.8X1_RECT"/>
 <part name="P16" library="Xevelabs" deviceset="PIN" device="_SMD_1X1_RECT" value="PIN_SMD_1X1_RECT"/>
-<part name="P17" library="Xevelabs" deviceset="PIN" device="_SMD_1X1_RECT" value="PIN_SMD_1X1_RECT"/>
-<part name="P18" library="Xevelabs" deviceset="PIN" device="_SMD_0.8X1_RECT" value="PIN_SMD_0.8X1_RECT"/>
+<part name="P17" library="Xevelabs" deviceset="PIN" device="_SMD_1X2" value="PIN_SMD_1X2"/>
 <part name="P8" library="Xevelabs" deviceset="PIN" device="_SMD_0.8X1_RECT" value="PIN_SMD_0.8X1_RECT"/>
 <part name="P9" library="Xevelabs" deviceset="PIN" device="_SMD_1X1_RECT" value="PIN_SMD_1X1_RECT"/>
 <part name="P10" library="Xevelabs" deviceset="PIN" device="_SMD_1X1_RECT" value="PIN_SMD_1X1_RECT"/>
-<part name="P11" library="Xevelabs" deviceset="PIN" device="_SMD_1X1_RECT" value="PIN_SMD_1X1_RECT"/>
+<part name="P11" library="Xevelabs" deviceset="PIN" device="_SMD_1X2" value="PIN_SMD_1X2"/>
 <part name="P12" library="Xevelabs" deviceset="PIN" device="_SMD_1X1_RECT" value="PIN_SMD_1X1_RECT"/>
 <part name="P13" library="Xevelabs" deviceset="PIN" device="_SMD_1X1_RECT" value="PIN_SMD_1X1_RECT"/>
@@
 <instance part="VDD3" gate="G$1" x="27.94" y="30.48"/>
 <instance part="VDD4" gate="G$1" x="71.12" y="17.78"/>
-<instance part="P1" gate="G$1" x="93.98" y="129.54" rot="MR0"/>
 <instance part="P2" gate="G$1" x="99.06" y="99.06" rot="MR0"/>
 <instance part="P3" gate="G$1" x="99.06" y="81.28" rot="MR0"/>
@@
 <instance part="P16" gate="G$1" x="114.3" y="119.38"/>
 <instance part="P17" gate="G$1" x="114.3" y="99.06"/>
-<instance part="P18" gate="G$1" x="114.3" y="81.28"/>
 <instance part="P8" gate="G$1" x="114.3" y="124.46"/>
 <instance part="P9" gate="G$1" x="114.3" y="104.14"/>
@@
 <instance part="VDD5" gate="G$1" x="96.52" y="60.96"/>
 <instance part="VDD6" gate="G$1" x="106.68" y="60.96"/>
-<instance part="P14" gate="G$1" x="99.06" y="134.62" rot="MR0"/>
+<instance part="P14" gate="G$1" x="109.22" y="134.62" rot="MR180"/>
 <instance part="C3" gate="G$1" x="15.24" y="15.24"/>
 </instances>
@@
 <segment>
 <pinref part="P3" gate="G$1" pin="1"/>
-<pinref part="P18" gate="G$1" pin="1"/>
 <wire x1="99.06" y1="81.28" x2="109.22" y2="81.28" width="0.1524" layer="91"/>
 <label x="101.6" y="81.28" size="1.778" layer="95"/>
 <pinref part="P10" gate="G$1" pin="1"/>
-<wire x1="109.22" y1="81.28" x2="114.3" y2="81.28" width="0.1524" layer="91"/>
 <wire x1="114.3" y1="86.36" x2="109.22" y2="86.36" width="0.1524" layer="91"/>
 <wire x1="109.22" y1="86.36" x2="109.22" y2="81.28" width="0.1524" layer="91"/>
@@
 </segment>
 </net>
-<net name="VDD_PASS" class="0">
-<segment>
-<pinref part="P1" gate="G$1" pin="1"/>
-<wire x1="93.98" y1="129.54" x2="101.6" y2="129.54" width="0.1524" layer="91"/>
-<wire x1="101.6" y1="129.54" x2="101.6" y2="134.62" width="0.1524" layer="91"/>
-<pinref part="P14" gate="G$1" pin="1"/>
-<wire x1="101.6" y1="134.62" x2="99.06" y2="134.62" width="0.1524" layer="91"/>
-<label x="101.6" y="129.54" size="1.778" layer="95"/>
-</segment>
-</net>
