File: elec/ssslidar_v1.0_blade_SIG_top.brd (EAGLE design)
At the start: 12 x 7 mm, 25 parts, among them P10 PIN_SMD_1X1_RECT, P11 PIN_SMD_1X2, P12 PIN_SMD_1X1_RECT, P13 PIN_SMD_1X1_RECT, P15 PIN_SMD_0.8X1_RECT, P16 PIN_SMD_1X1_RECT, P17 PIN_SMD_1X2, P18 PIN_SMD_0.8X1_RECT, P19 PIN_SMD_0.8X1_RECT, P2 PIN_SMD_1X1_RECT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

Commit message: Updated all libs.
Parts:
- turned P11 to 90 degrees
- turned P17 to 270 degrees
Changed lines of the file:
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@@
 <element name="P7" library="Xevelabs" package="PIN_SMD_0.8X1_RECT" value="PIN_SMD_0.8X1_RECT" x="5.2" y="0.75" rot="MR90"/>
 <element name="P16" library="Xevelabs" package="PIN_SMD_1X1_RECT" value="PIN_SMD_1X1_RECT" x="0.75" y="3.15" rot="R180"/>
-<element name="P17" library="Xevelabs" package="PIN_SMD_1X2" value="PIN_SMD_1X2" x="0.75" y="1.25" rot="MR0"/>
+<element name="P17" library="Xevelabs" package="PIN_SMD_1X2" value="PIN_SMD_1X2" x="0.75" y="1.25" rot="MR270"/>
 <element name="P9" library="Xevelabs" package="PIN_SMD_1X1_RECT" value="PIN_SMD_1X1_RECT" x="0.75" y="6.25"/>
 <element name="P10" library="Xevelabs" package="PIN_SMD_1X1_RECT" value="PIN_SMD_1X1_RECT" x="0.75" y="4.6" rot="MR180"/>
-<element name="P11" library="Xevelabs" package="PIN_SMD_1X2" value="PIN_SMD_1X2" x="0.75" y="1.25"/>
+<element name="P11" library="Xevelabs" package="PIN_SMD_1X2" value="PIN_SMD_1X2" x="0.75" y="1.25" rot="R90"/>
 <element name="P12" library="Xevelabs" package="PIN_SMD_1X1_RECT" value="PIN_SMD_1X1_RECT" x="0.75" y="4.6"/>
 <element name="P13" library="Xevelabs" package="PIN_SMD_1X1_RECT" value="PIN_SMD_1X1_RECT" x="0.75" y="3.15" rot="MR0"/>
@@
 <wire x1="0.85" y1="1.9" x2="0.85" y2="1.25" width="0.15" layer="16"/>
 <wire x1="0.85" y1="1.25" x2="0.75" y2="1.25" width="0.15" layer="16"/>
-<wire x1="0.85" y1="1.9" x2="0.85" y2="1.3" width="0.15" layer="1"/>
-<wire x1="0.85" y1="1.3" x2="0.85" y2="1.25" width="0.15" layer="1"/>
+<wire x1="0.85" y1="1.9" x2="0.85" y2="1.25" width="0.15" layer="1"/>
 <wire x1="0.85" y1="1.25" x2="0.75" y2="1.25" width="0.15" layer="1"/>
 <wire x1="0.9" y1="6.1" x2="0.75" y2="6.25" width="0.15" layer="1"/>
